Commit message: remote control

File: description/ros2_control/capstone.ros2_control.xacro (robot description, xacro)
@@ -6,9 +6,11 @@
         <plugin>diffdrive_arduino/DiffDriveArduinoHardware</plugin>
         <param name="left_wheel_name">left_wheel_joint</param>
+        <param name="right_wheel_name">right_wheel_joint</param>
         <param name="loop_rate">30</param>
-        <param name="device">/dev/ttyACM0</param>
+        <param name="device1">/dev/ttyACM0</param>
+        <param name="device2">/dev/ttyACM1</param>
         <param name="baud_rate">57600</param>
         <param name="timeout_ms">1000</param>
-        <param name="enc_counts_per_rev">3436</param>
+        <param name="enc_counts_per_rev">4096</param>
         <param name="pid_p">20</param>
         <param name="pid_d">12</param>
@@ -28,9 +30,11 @@
         <state_interface name="velocity"/>
       </joint>
-      <!-- <joint name="${prefix}right_wheel_joint">
+      <joint name="${prefix}right_wheel_joint">
         <command_interface name="velocity"/>
+            <param name="min">-10</param>
+            <param name="max">10</param>
         <state_interface name="position"/>
         <state_interface name="velocity"/>
-      </joint> -->
+      </joint>
     </ros2_control>
   </xacro:macro>

File: description/ros2_control/capstone_fake.ros2_control.xacro (robot description, xacro)
@@ -15,9 +15,9 @@
         <state_interface name="velocity"/>
       </joint>
-      <!-- <joint name="${prefix}right_wheel_joint">
+      <joint name="${prefix}right_wheel_joint">
         <command_interface name="velocity"/>
         <state_interface name="position"/>
         <state_interface name="velocity"/>
-      </joint> -->
+      </joint>
     </ros2_control>
   </xacro:macro>

File: description/ros2_control/capstone_gazebo.ros2_control copy.xacro (robot description, xacro)
@@ -24,6 +24,6 @@
     </joint>
     <gazebo>
-        <plugin name="gazebo_ros2_control" filename="libgazebo_ros2_control.so">
-        <parameters>$(find diffdrive_arduino)/config/capstone_controllers.yaml</parameters>
+      <plugin name="gazebo_ros2_control" filename="libgazebo_ros2_control.so">
+        <parameters>$(find diffdrive_arduino)/config/diff_drive_controller.yaml</parameters>
       </plugin>
     </gazebo>
