Commit message: 0424_update

File: description/ros2_control/capstone_two_arduino.ros2_control.xacro (robot description, xacro)
@@ -7,6 +7,7 @@
         <param name="left_wheel_name">left_wheel_joint</param>
         <param name="right_wheel_name">right_wheel_joint</param>
-        <param name="loop_rate">50</param>
-        <param name="device">/dev/ttyUSB0</param>
+        <param name="loop_rate">30</param>
+        <param name="device1">/dev/ttyACM0</param>
+        <param name="device2">/dev/ttyACM1</param>
         <param name="baud_rate">57600</param>
         <param name="timeout_ms">1000</param>
@@ -23,6 +24,6 @@
       <joint name="left_wheel_joint">
         <command_interface name="velocity">
-            <param name="min">-10</param>
-            <param name="max">10</param>
+          <param name="min">-1</param>
+          <param name="max">1</param>
         </command_interface>
         <state_interface name="position"/>
@@ -30,11 +31,11 @@
       </joint>
       <joint name="right_wheel_joint">
-        <command_interface name="velocity"/>
-            <param name="min">-10</param>
-            <param name="max">10</param>
+        <command_interface name="velocity">
+          <param name="min">-1</param>
+          <param name="max">1</param>
+        </command_interface>
         <state_interface name="position"/>
         <state_interface name="velocity"/>
       </joint>
-    </ros2_control>
   </xacro:macro>
 </robot>

File: description/urdf/capstone.urdf.xacro (robot description, xacro)
@@ -4,5 +4,5 @@
   <xacro:arg name="prefix" default="" />
   <xacro:arg name="use_gazebo" default="false"/>
-  <xacro:arg name="fake_hardware_" default="true"/>
+  <xacro:arg name="use_fake_hardware" default="true"/>
   <xacro:include filename="$(find diffdrive_arduino)/urdf/capstone_description.urdf.xacro" />
   <!-- Import Rviz colors -->

File: description/urdf/capstone_description.urdf.xacro (robot description, xacro)
@@ -2,79 +2,116 @@
 <robot xmlns:xacro="http://www.ros.org/wiki/xacro">
   <xacro:macro name="capstone" params="prefix">
-    <!-- Define the world link -->
-    <link name="${prefix}world"/>
-    <!-- Define the box -->
-    <link name="${prefix}box_link">
+    <link name="chassis">
+      <collision>
+        <origin xyz="-0.151427 -0 0.5" rpy="0 0 0"/>
+        <geometry>
+          <box size="2.01142 1 0.568726"/>
+        </geometry>
+      </collision>
+      <visual>
+        <origin xyz="-0.151427 -0 0.5" rpy="0 0 0"/>
+        <geometry>
+          <box size="2.01142 1 0.568726"/>
+        </geometry>
+      </visual>
+      <inertial>
+        <origin xyz="-0.151427 -0 0.5" rpy="0 0 0"/>
+        <mass value="1.14395"/>
+        <inertia
+          ixx="0.126164"
+          ixy="0.0"
+          ixz="0.0"
+          iyy="0.416519"
+          iyz="0.0"
+          izz="0.481014"/>
+      </inertial>
+    </link>
+    <joint name="left_wheel_joint" type="continuous">
+      <origin xyz="0.554283 0.625029 0.3" rpy="-1.5707 0 0"/>
+      <parent link="chassis"/>
+      <child link="left_wheel"/>
+      <axis xyz="0 0 1"/>
+      <dynamics damping="0.2"/>
+    </joint>
+    <!-- left wheel Link -->
+    <link name="left_wheel">
+      <collision>
+        <geometry>
+          <sphere radius="0.3"/>
+        </geometry>
+      </collision>
       <visual>
         <geometry>
-          <box size="0.1 0.1 0.1"/>
+          <sphere radius="0.3"/>
         </geometry>
       </visual>
+      <inertial>
+        <mass value="2"/>
+        <inertia ixx="0.145833"
+                ixy="0.0"
+                ixz="0.0"
+                iyy="0.145833"
+                iyz="0.0"
+                izz="0.125"/>
+      </inertial>
+    </link>
+    <joint name="right_wheel_joint" type="continuous">
+      <origin xyz="0.554283 -0.625029 0.3" rpy="-1.5707 0 0"/>
+      <parent link="chassis"/>
+      <child link="right_wheel"/>
+      <axis xyz="0 0 1"/>
+      <dynamics damping="0.2"/>
+    </joint>
+    <!-- right wheel Link -->
+    <link name="right_wheel">
       <collision>
         <geometry>
-          <box size="0.1 0.1 0.1"/>
+          <sphere radius="0.3"/>
         </geometry>
       </collision>
+      <visual>
+        <geometry>
+          <sphere radius="0.3"/>
+        </geometry>
+      </visual>
       <inertial>
-        <origin xyz="0 0 0" />
-        <mass value="1.0" />
-        <inertia ixx="0.001" ixy="0.0" ixz="0.0" iyy="0.001" iyz="0.0" izz="0.001"/>
+        <mass value="2"/>
+        <inertia ixx="0.145833"
+                ixy="0.0"
+                ixz="0.0"
+                iyy="0.145833"
+                iyz="0.0"
+                izz="0.125"/>
+        </inertial>
+    </link>
+    <joint name="caster_joint" type="fixed">
+      <origin xyz="-0.957138 -0 0.2" rpy="0 0 0"/>
+      <parent link="chassis"/>
+      <child link="caster"/>
+    </joint>
+    <!-- caster frontal wheel Link -->
+    <link name="caster">
+      <collision>
+        <geometry>
+          <sphere radius="0.2"/>
+        </geometry>
+      </collision>
+      <visual>
+        <geometry>
+          <sphere radius="0.2"/>
+        </geometry>
+      </visual>
+      <inertial>
+        <origin xyz="-0.957138 -0 0.2" rpy="0 0 0"/>
+        <mass value="0.005"/>
+        <inertia
+          ixx="0.1"
+          ixy="0.0"
+          ixz="0.0"
+          iyy="0.1"
+          iyz="0.0"
+          izz="0.1"/>
       </inertial>
     </link>
-    <!-- Define the stick -->
-    <link name="${prefix}stick_link">
-      <visual>
-        <geometry>
-          <cylinder length="0.1" radius="0.01"/>
-        </geometry>
-      </visual>
-      <collision>
-        <geometry>
-          <cylinder length="0.1" radius="0.01"/>
-        </geometry>
-      </collision>
-      <inertial>
-        <origin xyz="0 0 0.0" />
-        <mass value="0.1" />
-        <inertia ixx="0.0001" ixy="0.0" ixz="0.0" iyy="0.0001" iyz="0.0" izz="0.0001"/>
-      </inertial>
-    </link>
-    <!-- Define the box on the stick -->
-    <link name="${prefix}box_on_stick_link">
-      <visual>
-        <geometry>
-          <box size="0.05 0.05 0.01"/>
-        </geometry>
-      </visual>
-      <collision>
-        <geometry>
-          <box size="0.05 0.05 0.01"/>
-        </geometry>
-      </collision>
-      <inertial>
-        <origin xyz="0 0 0" />
-        <mass value="0.05" />
-        <inertia ixx="0.00001" ixy="0.0" ixz="0.0" iyy="0.00001" iyz="0.0" izz="0.00001"/>
-      </inertial>
-    </link>
-    <!-- Define the fixed joint connecting the box to the world -->
-    <joint name="${prefix}fixed_joint" type="fixed">
-      <parent link="${prefix}world"/>
-      <child link="${prefix}box_link"/>
-      <origin xyz="0 0 0.1"/>
-    </joint>
-    <!-- Define the revolute joint connecting the stick to the box -->
-    <joint name="${prefix}left_wheel_joint" type="continuous">
-      <parent link="${prefix}box_link"/>
-      <child link="${prefix}stick_link"/>
-      <origin xyz="0 0 0.1"/>
-      <axis xyz="0 0 1"/>
-    </joint>
-    <!-- Define the fixed joint connecting the box on the stick -->
-    <joint name="${prefix}fixed_joint_box_on_stick" type="fixed">
-      <parent link="${prefix}stick_link"/>
-      <child link="${prefix}box_on_stick_link"/>
-      <origin xyz="0.025 0 0.1"/>
-    </joint>
   </xacro:macro>
 </robot>
